File: kicad_vectron_65_plus/kicad_vectron_65_plus.kicad_pcb (KiCad board)
At the start: 4 copper layers, 131.1 x 79.4 mm, 48 parts, among them J1 Power, J2 Power, J3 VIA 1 Ports, J4 Conn_01x16_Male, J5 PS/2 Keyboard, J6 Power, J7 Power, SW1 SW_Push_Dual, U1 W65C02SxP, U10 SN74LS08N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

Commit message: Save progress on PCB.
Parts:
- moved R1 78.4 mm to (63.6, 43.8), turned to 180 degrees
- moved J2 44.4 mm to (122.5, 34.0), turned to 90 degrees
- moved J3 11.2 mm to (166.8, 40.0)
- moved R3 2.59 mm to (69.1, 66.8)
- moved C16 0.14 mm to (157.0, 41.2)
Routing:
- net Net-(U1-Pad27): track 0.00 -> 252.8 mm, vias 0 -> 10
- net Net-(U1-Pad28): track 0.00 -> 247.6 mm, vias 0 -> 8
- net Net-(U1-Pad34): track 0.00 -> 242.1 mm, vias 0 -> 1
- net Net-(U1-Pad30): track 0.00 -> 229.8 mm, vias 0 -> 4
- net Net-(U1-Pad31): track 0.00 -> 220.3 mm, vias 0 -> 6
- net Net-(U1-Pad29): track 0.00 -> 210.9 mm, vias 0 -> 9
- net Net-(U1-Pad32): track 0.00 -> 201.3 mm, vias 0 -> 5
- net Net-(U1-Pad12): track 0.00 -> 200.2 mm, vias 0 -> 5
- net Net-(U1-Pad33): track 0.00 -> 198.8 mm, vias 0 -> 5
- net Net-(U1-Pad11): track 0.00 -> 181.4 mm, vias 0 -> 8
- net Net-(U1-Pad15): track 0.00 -> 180.5 mm, vias 0 -> 5
- net Net-(U1-Pad4): track 0.00 -> 171.0 mm, vias 0 -> 5
- net Net-(U1-Pad10): track 0.00 -> 167.7 mm, vias 0 -> 10
- net Net-(U1-Pad39): track 0.00 -> 166.9 mm, vias 0 -> 2
- net Net-(U11-Pad6): track 0.00 -> 144.4 mm, vias 0 -> 4
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
Commit message: Save progress on PCB.
Routing:
- net Net-(U1-Pad9): track 128.3 -> 223.8 mm, vias 4 -> 7
- net Net-(U1-Pad17): track 101.3 -> 181.6 mm, vias 2 -> 4
- net Net-(U1-Pad19): track 55.8 -> 132.9 mm
- net Net-(U1-Pad26): track 112.0 -> 186.4 mm, vias 4 -> 5
- net Net-(U1-Pad20): track 70.8 -> 125.6 mm, vias 3 -> 4
- net Net-(U1-Pad14): track 99.2 -> 135.2 mm, vias 0 -> 3
- net Net-(U1-Pad18): track 65.6 -> 95.1 mm, vias 1 -> 4
- net Net-(R5-Pad1): track 0.00 -> 3.34 mm
- net Net-(R8-Pad1): track 0.00 -> 3.19 mm
- net +5V: track 0.00 -> 2.84 mm
- net Net-(U1-Pad30): track 229.8 -> 231.8 mm, vias 4 -> 7
- net Net-(U1-Pad10): track 167.7 -> 166.4 mm, vias 10 -> 9

Commit message: Save progress on PCB.
Parts:
- renumbered SW1 to Reset
Other:
- board text added: "+"
- board text added: "10K"
- board text added: "3.3K"
- board text added: "5"
- board text added: "5.1K"
- board text added: "5V"
- board text added: "6"
- board text added: "6502"
- board text added: "7404"
- board text added: "7408"
- board text added: "7432"
- board text added: "74682"
- board text added: "G"
- board text added: "Keyboard"
- board text added: "Nick Bild May 2022 v1.0"
- board text added: "PA0"
- board text added: "PB7"
- board text added: "Plus"
- board text added: "Power"
- board text added: "RAM"
- board text added: "ROM"
- board text added: "S"
- board text added: "V"
- board text added: "VIA 1"
- board text added: "VIA 1 Ports"
- board text added: "VIA 2"
- board text added: "VIA 2 Ports"
- board text added: "c"
- board text added: "e"
- board text added: "github.com/nickbild/vectron_65_plus"
- board text added: "n"
- board text added: "o"
- board text added: "r"
- board text added: "t"
