File: kicad_vectron_65_plus/kicad_vectron_65_plus.sch (KiCad schematic (older format))
At the start: 31 parts

Commit message: Update schematic.
Parts:
- added R? (x4): 3.3K, symbol Device:R
Connections:
- net at U?.10 (A1): now also U?.37 (RS1), U?.9 (A1)
- net at U?.11 (A2): now also U?.36 (RS2), U?.8 (A2)
- net at U?.12 (A3): now also U?.35 (RS3), U?.7 (A3)
- net at U?.13 (A4): now also U?.3 (Q0), U?.6 (A4)
- net at U?.14 (A5): now also U?.5 (A5), U?.5 (Q1)
- net at U?.15 (A6): now also U?.4 (A6), U?.7 (Q2)
- net at U?.16 (A7): now also U?.3 (A7), U?.9 (Q3)
- net at U?.17 (A8): now also U?.25 (A8), U?.3 (Q0)
- net at U?.18 (A9): now also U?.24 (A9), U?.5 (Q1)
- net at U?.19 (A10): now also U?.21 (A10), U?.7 (Q2)
- net at U?.2 (RDY): now also R?.1
- net at U?.20 (A11): now also U?.23 (A11), U?.9 (Q3)
- net GND: now reaches U?.21 (VSS)
- net GND: now also X?.7 (GND)
- net at U?.22 (A12): now also U?.12 (Q4), U?.2 (A12)
- net at U?.23 (A13): now also U?.14 (Q5), U?.26 (A13)
- net at U?.24 (A14): now also U?.1 (A14), U?.16 (Q6)
- net at U?.25 (A15): now also U?.18 (Q7), U?.5 (3A)
- net at U?.26 (D7): now also U?.19 (D7), U?.26 (D7)
- net at U?.27 (D6): now also U?.18 (D6), U?.27 (D6)
- net at U?.28 (D5): now also U?.17 (D5), U?.28 (D5)
- net at U?.29 (D4): now also U?.16 (D4), U?.29 (D4)
- net at U?.30 (D3): now also U?.15 (D3), U?.30 (D3)
- net at U?.31 (D2): now also U?.13 (D2), U?.31 (D2)
- net at U?.32 (D1): now also U?.12 (D1), U?.32 (D1)
- net at U?.33 (D0): now also U?.11 (D0), U?.33 (D0)
- net at U?.34 (R/~W): now also U?.1 (1A)
- net at U?.36 (BE): now also R?.1
- net at U?.37 (ϕ0): now also X?.8 (OUT)
- net +5V: now reaches U?.38 (~SO)
- net +5V: now also U?.8 (VDD), X?.14 (Vcc), R?.2, R?.2, R?.2, R?.2
- net at U?.39 (ϕ2): now also U?.1 (1A), U?.25 (ϕ2)
- net at U?.4 (~IRQ): now also U?.21 (~IRQ)
- net at U?.40 (~RES): now also SW?.2, U?.34 (~RES), R?.1
- net at U?.6 (~NMI): now also R?.1
- net at U?.9 (A0): now also U?.10 (A0), U?.38 (RS0)
Other:
- moved on the sheet: C?, U?

Commit message: Save progress on schematic.
Connections:
- net +5V: now also U?.27 (~WE), U?.28 (VCC), U?.28 (VCC)
- net GND: now also U?.14 (GND), U?.14 (GND), U?.22 (~OE)
- net at U?.10 (A1), U?.37 (RS1), U?.9 (A1): now also U?.9 (A1)
- net at U?.11 (A2), U?.36 (RS2), U?.8 (A2): now also U?.8 (A2)
- net at U?.12 (A3), U?.35 (RS3), U?.7 (A3): now also U?.7 (A3)
- net at U?.13 (A4), U?.3 (Q0), U?.6 (A4): now also U?.18 (Q7), U?.6 (A4)
- net at U?.14 (A5), U?.5 (A5), U?.5 (Q1): now also U?.16 (Q6), U?.5 (A5)
- net at U?.15 (A6), U?.4 (A6), U?.7 (Q2): now also U?.14 (Q5), U?.4 (A6)
- net at U?.16 (A7), U?.3 (A7), U?.9 (Q3): now also U?.12 (Q4), U?.3 (A7)
- net at U?.17 (A8), U?.25 (A8), U?.3 (Q0): now also U?.25 (A8)
- net at U?.18 (A9), U?.24 (A9), U?.5 (Q1): now also U?.24 (A9)
- net at U?.19 (A10), U?.21 (A10), U?.7 (Q2): now also U?.21 (A10)
- net at U?.20 (A11), U?.23 (A11), U?.9 (Q3): now also U?.23 (A11)
- net at U?.12 (Q4), U?.2 (A12), U?.22 (A12): now also U?.2 (A12)
- net at U?.14 (Q5), U?.23 (A13), U?.26 (A13): now also U?.26 (A13)
- net at U?.1 (A14), U?.16 (Q6), U?.24 (A14): now also U?.1 (A14)
- net at U?.19 (D7), U?.26 (D7), U?.26 (D7): now also U?.19 (D7)
- net at U?.18 (D6), U?.27 (D6), U?.27 (D6): now also U?.18 (D6)
- net at U?.17 (D5), U?.28 (D5), U?.28 (D5): now also U?.17 (D5)
- net at U?.16 (D4), U?.29 (D4), U?.29 (D4): now also U?.16 (D4)
- net at U?.15 (D3), U?.30 (D3), U?.30 (D3): now also U?.15 (D3)
- net at U?.13 (D2), U?.31 (D2), U?.31 (D2): now also U?.13 (D2)
- net at U?.12 (D1), U?.32 (D1), U?.32 (D1): now also U?.12 (D1)
- net at U?.11 (D0), U?.33 (D0), U?.33 (D0): now also U?.11 (D0)
- net at U?.10 (A0), U?.38 (RS0), U?.9 (A0): now also U?.10 (A0)
- net at U?.20 (~CS): now also U?.6 (3Y)
- net at U?.20 (~CS): now also U?.1 (*P>Q)
- net at U?.22 (~OE): now also U?.2 (1Y)
- net at U?.27 (~WE): now also U?.4 (2Y)
Other:
- moved on the sheet: C?

Commit message: Save progress on schematic.
Parts:
- added C?: C, symbol Device:C
- added J? (x4): Power, symbol Connector:Conn_01x05_Male
- added J?: VIA 1 Ports, symbol Connector:Conn_01x16_Male
- added J?: Conn_01x16_Male, symbol Connector:Conn_01x16_Male
- added R? (x4): 10K, symbol Device:R
- added R? (x2): 5.1K, symbol Device:R
- U?: value W65C22SxP -> VIA 1
- U?: value W65C22SxP -> VIA 2
Connections:
- net +5V: now also C?.1, C?.1, C?.1, C?.1, C?.1, C?.1, C?.1, C?.1, C?.1, C?.1, C?.1, C?.1, C?.1, C?.1, C?.1, C?.1, J?.4, U?.11 (P4), U?.11 (P4), U?.11 (P4), U?.13 (P5), U?.13 (P5), U?.13 (P5), U?.14 (VCC), U?.14 (VCC), U?.14 (VCC), U?.15 (P6), U?.15 (P6), U?.15 (P6), U?.17 (P7), U?.2 (P0), U?.20 (VCC), U?.20 (VCC), U?.20 (VCC), U?.20 (VCC), U?.20 (VCC), U?.20 (VCC), U?.4 (P1), U?.6 (P2), U?.8 (P3), C?.1, J?.1 (Pin_1), J?.1 (Pin_1), J?.1 (Pin_1), J?.1 (Pin_1), J?.2 (Pin_2), J?.2 (Pin_2), J?.2 (Pin_2), J?.2 (Pin_2), R?.1, R?.2
- net GND: now also C?.2, C?.2, C?.2, C?.2, C?.2, C?.2, C?.2, C?.2, C?.2, C?.2, C?.2, C?.2, C?.2, C?.2, C?.2, C?.2, J?.3, U?.1 (VSS), U?.1 (VSS), U?.10 (GND), U?.10 (GND), U?.10 (GND), U?.10 (GND), U?.11 (P4), U?.13 (P5), U?.15 (P6), U?.17 (P7), U?.17 (P7), U?.17 (P7), U?.2 (P0), U?.2 (P0), U?.2 (P0), U?.3 (Q0), U?.3 (Q0), U?.4 (P1), U?.4 (P1), U?.4 (P1), U?.5 (Q1), U?.5 (Q1), U?.6 (P2), U?.6 (P2), U?.6 (P2), U?.7 (GND), U?.7 (GND), U?.7 (GND), U?.7 (Q2), U?.7 (Q2), U?.8 (P3), U?.8 (P3), U?.8 (P3), U?.9 (Q3), U?.9 (Q3), C?.2, J?.3 (Pin_3), J?.3 (Pin_3), J?.3 (Pin_3), J?.3 (Pin_3), J?.4 (Pin_4), J?.4 (Pin_4), J?.4 (Pin_4), J?.4 (Pin_4), J?.5 (Pin_5), J?.5 (Pin_5), J?.5 (Pin_5), J?.5 (Pin_5), R?.1, R?.1, R?.2, R?.2
- net at U?.10 (A1), U?.37 (RS1), U?.9 (A1)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: now also U?.16 (Q6), U?.37 (RS1)
- net at U?.11 (A2), U?.36 (RS2), U?.8 (A2)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: now also U?.14 (Q5), U?.36 (RS2)
- net at U?.12 (A3), U?.35 (RS3), U?.7 (A3)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: now also U?.12 (Q4), U?.35 (RS3)
- net at U?.13 (A4), U?.18 (Q7), U?.3 (Q0)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: now also U?.18 (Q7)
- net at U?.14 (A5), U?.16 (Q6), U?.5 (A5)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: now also U?.16 (Q6)
- net at U?.14 (Q5), U?.15 (A6), U?.4 (A6)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: now also U?.14 (Q5)
- net at U?.12 (Q4), U?.16 (A7), U?.3 (A7)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: now also U?.12 (Q4)
- net at U?.19 (D7), U?.19 (D7), U?.26 (D7)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: now also U?.26 (D7)
- net at U?.18 (D6), U?.18 (D6), U?.27 (D6)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: now also U?.27 (D6)
- net at U?.17 (D5), U?.17 (D5), U?.28 (D5)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: now also U?.28 (D5)
- net at U?.16 (D4), U?.16 (D4), U?.29 (D4)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: now also U?.29 (D4)
- net at U?.15 (D3), U?.15 (D3), U?.30 (D3)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: now also U?.30 (D3)
- net at U?.13 (D2), U?.13 (D2), U?.31 (D2)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: now also U?.31 (D2)
- net at U?.12 (D1), U?.12 (D1), U?.32 (D1)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: now also U?.32 (D1)
- net at U?.11 (D0), U?.11 (D0), U?.33 (D0)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: now also U?.33 (D0)
- net at U?.1 (1A), U?.34 (R/~W): now also U?.22 (R/~W), U?.22 (R/~W)
- net at U?.1 (1A), U?.25 (ϕ2), U?.39 (ϕ2): now also U?.12 (4A), U?.25 (ϕ2)
- net at R?.1, SW?.2, U?.34 (~RES)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: now also U?.34 (~RES)
- net at U?.10 (A0), U?.10 (A0), U?.38 (RS0)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: now also U?.18 (Q7), U?.38 (RS0)
- net at U?.10 (PB0): now also J?.9 (Pin_9) (x2)
- net at U?.11 (PB1): now also J?.10 (Pin_10) (x2)
- net at U?.12 (PB2): now also J?.11 (Pin_11) (x2)
- net at U?.13 (PB3): now also J?.12 (Pin_12) (x2)
- net at U?.14 (PB4): now also J?.13 (Pin_13)
- net at U?.15 (PB5): now also J?.14 (Pin_14)
- net at U?.16 (PB6): now also J?.15 (Pin_15) (x2)
- net at U?.17 (PB7): now also J?.16 (Pin_16) (x2)
- net at U?.18 (CB1): now also R?.1
- net at U?.19 (CB2): now also R?.1
- net at U?.2 (PA0): now also J?.1 (Pin_1) (x2)
- net at U?.23 (~CS2): now also U?.11 (4Y), U?.9 (4A)
- net at U?.24 (CS1): now also U?.8 (4Y)
- net at U?.3 (PA1): now also J?.2 (Pin_2) (x2)
- net at U?.39 (CA2): now also R?.2
- net at U?.4 (PA2): now also J?.3 (Pin_3) (x2)
- net at U?.40 (CA1): now also R?.2
- net at U?.5 (PA3): now also J?.4 (Pin_4) (x2)
- net at U?.6 (PA4): now also J?.5 (Pin_5) (x2)
- net at U?.7 (PA5): now also J?.6 (Pin_6) (x2)
- net at U?.8 (PA6): now also J?.7 (Pin_7) (x2)
- net at U?.9 (PA7): now also J?.8 (Pin_8) (x2)
- net at U?.14 (PB4): now also J?.5, J?.13 (Pin_13), R?.1
- net at U?.15 (PB5): now also J?.1, J?.14 (Pin_14), R?.2
- net at U?.23 (~CS2): now also U?.11 (5A), U?.6 (2Y)
- net at U?.24 (CS1): now also U?.10 (5Y)
- net at U?.2 (1Y), U?.22 (~OE): now also U?.2 (1B)
- net at U?.12 (6Y): now also U?.13 (4B)
- net at U?.13 (6A): now also U?.8 (3Y)
- net at U?.3 (2A): now also U?.3 (1Y)
- net at U?.19 (*P=Q): now also U?.4 (2A)
- net at U?.19 (*P=Q): now also U?.12 (4A), U?.5 (2B), U?.9 (3A)
- net at U?.19 (*P=Q): now also U?.13 (4B)
- net at U?.10 (3B): now also U?.19 (*P=Q)
Other:
- moved on the sheet: C?

Commit message: Save progress on schematic.
Parts:
- C1, C10, C11, C12, C13, C14, C15, C3, C4, C5, C6, C7, C8, C9: renamed from C?; footprint (none) -> Capacitor_THT:C_Disc_D3.0mm_W2.0mm_P2.50mm
- C16, C17, C2: renamed from C?; footprint (none) -> Capacitor_THT:CP_Radial_D8.0mm_P5.00mm
- J1, J2, J6, J7: renamed from J?; footprint (none) -> Connector_PinHeader_2.54mm:PinHeader_1x05_P2.54mm_Vertical
- J3, J4: renamed from J?; footprint (none) -> Connector_PinHeader_2.54mm:PinHeader_1x16_P2.54mm_Vertical
- J5: renamed from J?; value 5750071-1 -> PS/2 Keyboard; footprint CONN_5750071-1_TYC -> 5750071-1:5750071-1
- R1, R10, R2, R3, R4, R5, R6, R7, R8, R9: renamed from R?; footprint (none) -> Resistor_THT:R_Axial_DIN0204_L3.6mm_D1.6mm_P5.08mm_Horizontal
- SW1: renamed from SW?; footprint (none) -> Button_Switch_THT:SW_TH_Tactile_Omron_B3F-10xx
- U1, U2, U5: renamed from U?; footprint (none) -> Package_DIP:DIP-40_W15.24mm
- U10, U11, U9: renamed from U?; footprint DIP794W45P254L1969H508Q14 -> Package_DIP:DIP-14_W7.62mm
- U12, U4, U7, U8: renamed from U?; footprint N20 -> Package_DIP:DIP-20_W7.62mm
- U3, U6: renamed from U?; footprint (none) -> Package_DIP:DIP-28_W15.24mm
- X1: renamed from X?; value CXO_DIP14 -> 8 MHz
Connections:
- net GND: now also SW1.3, SW1.4

Commit message: Mirror image for PS/2 connection.
Parts:
- J5: symbol 2022-05-02_22-16-01:5750071-1 -> kicad_vectron_65_plus-rescue:5750071-1-2022-05-02_22-16-01
Connections:
- net +5V: now also J5.3; no longer J5.4
- net GND: now also J5.4; no longer J5.3
- net at J4.13 (Pin_13), R9.1, U5.14 (PB4): now also J5.6; no longer J5.5
- net at J4.14 (Pin_14), R10.2, U5.15 (PB5): now also J5.2; no longer J5.1
Changed lines of the file:
@@
 $EndComp
 $Comp
-L 2022-05-02_22-16-01:5750071-1 J5
-U 1 1 6272E838
-P 9150 14900
-F 0 "J5" H 9678 14703 60  0000 L CNN
-F 1 "PS/2 Keyboard" H 9678 14597 60  0000 L CNN
-F 2 "5750071-1:5750071-1" H 9550 14640 60  0001 C CNN
-F 3 "" H 9150 14900 60  0000 C CNN
-	1    9150 14900
-	1    0    0    -1
-$EndComp
-$Comp
 L Device:CP C2
 U 1 1 6273A754
@@
 $EndComp
 Wire Wire Line
-	9150 15100 8750 15100
-Wire Wire Line
 	8750 15100 8750 14500
 Wire Wire Line
@@
 Wire Wire Line
 	8700 13100 8700 15300
-Wire Wire Line
-	8700 15400 9150 15400
-$Comp
-L power:+5V #PWR057
-U 1 1 6368985B
-P 9150 14900
-F 0 "#PWR057" H 9150 14750 50  0001 C CNN
-F 1 "+5V" H 9165 15073 50  0000 C CNN
-F 2 "" H 9150 14900 50  0001 C CNN
-F 3 "" H 9150 14900 50  0001 C CNN
-	1    9150 14900
-	1    0    0    -1
-$EndComp
-$Comp
-L power:GND #PWR058
-U 1 1 63689EDF
-P 9150 15200
-F 0 "#PWR058" H 9150 14950 50  0001 C CNN
-F 1 "GND" V 9155 15072 50  0000 R CNN
-F 2 "" H 9150 15200 50  0001 C CNN
-F 3 "" H 9150 15200 50  0001 C CNN
-	1    9150 15200
-	0    1    1    0
-$EndComp
 $Comp
 L power:+5V #PWR015
@@
 	1    0    0    -1
 $EndComp
+Wire Wire Line
+	8750 15100 8850 15100
+Wire Wire Line
+	8850 15100 8850 15000
+Wire Wire Line
+	8700 15400 8850 15400
+Wire Wire Line
+	8850 15400 8850 15300
+Wire Wire Line
+	8850 15300 9150 15300
+Wire Wire Line
+	8850 15000 9150 15000
+$Comp
+L power:+5V #PWR?
+U 1 1 62F0BBCA
+P 9150 15200
+F 0 "#PWR?" H 9150 15050 50  0001 C CNN
+F 1 "+5V" V 9165 15328 50  0000 L CNN
+F 2 "" H 9150 15200 50  0001 C CNN
+F 3 "" H 9150 15200 50  0001 C CNN
+	1    9150 15200
+	0    -1   -1   0
+$EndComp
+$Comp
+L kicad_vectron_65_plus-rescue:5750071-1-2022-05-02_22-16-01 J5
+U 1 1 6272E838
+P 9150 14900
+F 0 "J5" H 9678 14703 60  0000 L CNN
+F 1 "PS/2 Keyboard" H 9678 14597 60  0000 L CNN
+F 2 "5750071-1:5750071-1" H 9550 14640 60  0001 C CNN
+F 3 "" H 9150 14900 60  0000 C CNN
+	1    9150 14900
+	1    0    0    -1
+$EndComp
+$Comp
+L power:GND #PWR?
+U 1 1 62F8D9C3
+P 9150 14900
+F 0 "#PWR?" H 9150 14650 50  0001 C CNN
+F 1 "GND" H 9155 14727 50  0000 C CNN
+F 2 "" H 9150 14900 50  0001 C CNN
+F 3 "" H 9150 14900 50  0001 C CNN
+	1    9150 14900
+	-1   0    0    1
+$EndComp
 $EndSCHEMATC
